Commit message: Add laser scanner

File: gazebo_example/models/xacro/example_robot.urdf.xacro (robot description, xacro)
@@ -34,4 +34,66 @@
       </collision>
     </link>
+    <!-- hokuyo -->
+    <joint name="hokuyo_joint" type="fixed">
+       <axis xyz="0 1 0" />
+       <origin xyz="0 0 -0.3" rpy="0 1.57 0"/>
+       <parent link="${name}_link"/>
+       <child link="hokuyo_link"/>
+     </joint>
+    <!-- Hokuyo Laser -->
+    <link name="hokuyo_link">
+    <collision>
+         <origin xyz="0 0 0" rpy="0 0 0"/>
+         <geometry>
+             <box size="0.1 0.1 0.1"/>
+         </geometry>
+    </collision>
+    <visual>
+     <origin xyz="0 0 0" rpy="0 0 0"/>
+     <geometry>
+       <box size="0.1 0.1 0.1"/>
+     </geometry>
+    </visual>
+    <inertial>
+     <mass value="1e-5" />
+     <origin xyz="0 0 0" rpy="0 0 0"/>
+     <inertia ixx="1e-6" ixy="0" ixz="0" iyy="1e-6" iyz="0" izz="1e-6" />
+    </inertial>
+  </link>
+  <gazebo reference="hokuyo_link">
+    <sensor type="ray" name="head_hokuyo_sensor">
+      <pose>0 0 0 0 0 0</pose>
+      <visualize>true</visualize>
+      <update_rate>40</update_rate>
+      <ray>
+        <scan>
+          <horizontal>
+            <samples>720</samples>
+            <resolution>1</resolution>
+            <min_angle>-0.570796</min_angle>
+            <max_angle>0.570796</max_angle>
+          </horizontal>
+        </scan>
+        <range>
+          <min>0.10</min>
+          <max>30.0</max>
+          <resolution>0.01</resolution>
+        </range>
+        <noise>
+          <type>gaussian</type>
+          <!-- Noise parameters based on published spec for Hokuyo laser
+               achieving "+-30mm" accuracy at range < 10m.  A mean of 0.0m and
+               stddev of 0.01m will put 99.7% of samples within 0.03m of the true
+               reading. -->
+          <mean>0.0</mean>
+          <stddev>0.01</stddev>
+        </noise>
+      </ray>
+      <plugin name="gazebo_ros_head_hokuyo_controller" filename="libgazebo_ros_laser.so">
+        <topicName>/plane/laser/scan</topicName>
+        <frameName>hokuyo_link</frameName>
+      </plugin>
+    </sensor>
+  </gazebo>
   </xacro:macro>
   <xacro:plane_xacro name="$(arg robot_name)" />
